Commit message: Changes for aernova

File: kuka_kr300_support/urdf/kr300r2700_2_macro.xacro (robot description, xacro)
@@ -154,5 +154,5 @@
       <child link="${prefix}link_2"/>
       <axis xyz="0 1 0"/>
-      <limit lower="${radians(-55)}" upper="${radians(85)}" effort="0" velocity="${radians(101)}"/>
+      <limit lower="${radians(-50)}" upper="${radians(85)}" effort="0" velocity="${radians(101)}"/>
     </joint>
     <joint name="${prefix}joint_a3" type="revolute">
