Commit message: Update  changes to aernnova

File: kuka_kr120_support/urdf/kr120r2500pro.xacro (robot description, xacro)
@@ -1,3 +1,3 @@
-<?xml version="1.0"?>
+ g<?xml version="1.0"?>
 <!--Generates a urdf from the macro in kr120r2500pro_macro.xacro -->
 <robot name="kuka_kr120r2500pro" xmlns:xacro="http://wiki.ros.org/xacro">

File: kuka_kr180_support/urdf/kr180r3500_ultra_k_macro.xacro (robot description, xacro)
@@ -157,9 +157,9 @@
     </joint>
     <joint name="${prefix}joint_a3" type="revolute">
-      <origin xyz="0 -0.168 1.35" rpy="0 0 0"/>
+      <origin xyz="1.35 -0.168 0" rpy="0 0 0"/>
       <parent link="${prefix}link_2"/>
       <child link="${prefix}link_3"/>
       <axis xyz="0 1 0"/>
-      <limit lower="${radians(-210)}" upper="${radians(65)}" effort="0" velocity="${radians(107)}"/>
+      <limit lower="${radians(-120)}" upper="${radians(155)}" effort="0" velocity="${radians(107)}"/>
     </joint>
     <joint name="${prefix}joint_a4" type="revolute">
