Commit message: Update collisio meshes

File: kuka_kl4000_support/urdf/kl4000standard.xacro (robot description, xacro)
@@ -1,5 +1,6 @@
 <?xml version="1.0"?>
 <robot name="kuka_kl4000" xmlns:xacro="http://wiki.ros.org/xacro">
+  <xacro:arg name="prefix" default=""/>
   <xacro:include filename="$(find kuka_kl4000_support)/urdf/kl4000standard_macro.xacro"/>
-  <xacro:kuka_kl4000standard prefix=""/>
+  <xacro:kuka_kl4000standard prefix="$(arg prefix)"/>
 </robot>

File: kuka_kl4000_support/urdf/kl4000standard_macro.xacro (robot description, xacro)
@@ -44,5 +44,5 @@
     <link name="${prefix}flange"/>
     <!-- joints -->
-    <joint name="${prefix}joint_l1" type="prismatic">
+    <joint name="${prefix}joint_e1" type="prismatic">
       <origin xyz="0 0 0" rpy="0 0 0"/>
       <parent link="${prefix}base_link"/>
