Commit message: Fix tool0 placement

File: kuka_kl4000_support/urdf/kl4000standard_macro.xacro (robot description, xacro)
@@ -68,5 +68,5 @@
       <parent link="${prefix}flange"/>
       <child link="${prefix}tool0"/>
-      <origin xyz="0 0 0" rpy="0 ${radians(90)} 0"/>
+      <origin xyz="0 0 0" rpy="0 0 0"/>
     </joint>
     <!-- rename 'Link1' to 'link_1', maintain bw-compatibility -->

Commit message: Fix flange placement

File: kuka_kl4000_support/urdf/kl4000standard_macro.xacro (robot description, xacro)
@@ -54,5 +54,5 @@
       <parent link="${prefix}link_1"/>
       <child link="${prefix}flange"/>
-      <origin xyz="0 0 0.7" rpy="0 0 0"/>
+      <origin xyz="0 0 0.69" rpy="0 0 0"/>
     </joint>
     <!-- ROS base_link to KUKA $ROBROOT coordinate system transform -->

Commit message: Incorporate new meshes from aernnova

File: kuka_kl4000_support/urdf/kl4000standard_macro.xacro (robot description, xacro)
@@ -12,5 +12,5 @@
         <origin xyz="0 0 0" rpy="0 0 0"/>
         <geometry>
-          <mesh filename="package://kuka_kl4000_support/meshes/kl4000standard/visual/base_link.dae"/>
+          <mesh filename="package://kuka_kl4000_support/meshes/kl4000standard/visual/base_link_aernnova.dae"/>
         </geometry>
       </visual>

File: kuka_kr180_support/urdf/kr180r3500_ultra_k_macro.xacro (robot description, xacro)
@@ -69,5 +69,5 @@
         <origin xyz="0 0 0" rpy="0 0 0"/>
         <geometry>
-          <mesh filename="package://kuka_kr180_support/meshes/kr180r3500_ultra_k/visual/link_3.dae"/>
+          <mesh filename="package://kuka_kr180_support/meshes/kr180r3500_ultra_k/visual/link_3_aernnova.dae"/>
         </geometry>
         <material name="">
@@ -78,5 +78,5 @@
         <origin xyz="0 0 0" rpy="0 0 0"/>
         <geometry>
-          <mesh filename="package://kuka_kr180_support/meshes/kr180r3500_ultra_k/collision/link_3.stl"/>
+          <mesh filename="package://kuka_kr180_support/meshes/kr180r3500_ultra_k/collision/link_3_aernnova.stl"/>
         </geometry>
       </collision>
@@ -129,11 +129,11 @@
         <origin xyz="0 0 0" rpy="0 0 0"/>
         <geometry>
-          <mesh filename="package://kuka_kr180_support/meshes/kr180r3500_ultra_k/visual/link_6.dae"/>
-        </geometry>
-      </visual>
-      <collision>
-        <origin xyz="0 0 0" rpy="0 0 0"/>
-        <geometry>
-          <mesh filename="package://kuka_kr180_support/meshes/kr180r3500_ultra_k/collision/link_6.stl"/>
+          <mesh filename="package://kuka_kr180_support/meshes/kr180r3500_ultra_k/visual/link_6_aernnova.dae"/>
+        </geometry>
+      </visual>
+      <collision>
+        <origin xyz="0 0 0" rpy="0 0 0"/>
+        <geometry>
+          <mesh filename="package://kuka_kr180_support/meshes/kr180r3500_ultra_k/collision/link_6_aernnova.stl"/>
         </geometry>
       </collision>
