Commit message: Fix limits of joint 2

File: kuka_kr180_support/urdf/kr180r3500_ultra_k_macro.xacro (robot description, xacro)
@@ -154,5 +154,5 @@
       <child link="${prefix}link_2"/>
       <axis xyz="0 1 0"/>
-      <limit lower="${radians(-30)}" upper="${radians(160)}" effort="0" velocity="${radians(101)}"/>
+      <limit lower="${radians(-120)}" upper="${radians(70)}" effort="0" velocity="${radians(101)}"/>
     </joint>
     <joint name="${prefix}joint_a3" type="revolute">

Commit message: Fix direction of axes

File: kuka_kr180_support/urdf/kr180r3500_ultra_k_macro.xacro (robot description, xacro)
@@ -146,5 +146,5 @@
       <parent link="${prefix}base_link"/>
       <child link="${prefix}link_1"/>
-      <axis xyz="0 0 1"/>
+      <axis xyz="0 0 -1"/>
       <limit lower="${radians(-185)}" upper="${radians(185)}" effort="0" velocity="${radians(105)}"/>
     </joint>
@@ -167,5 +167,5 @@
       <parent link="${prefix}link_3"/>
       <child link="${prefix}link_4"/>
-      <axis xyz="1 0 0"/>
+      <axis xyz="-1 0 0"/>
       <limit lower="${radians(-350)}" upper="${radians(350)}" effort="0" velocity="${radians(179)}"/>
     </joint>
@@ -181,5 +181,5 @@
       <parent link="${prefix}link_5"/>
       <child link="${prefix}link_6"/>
-      <axis xyz="1 0 0"/>
+      <axis xyz="-1 0 0"/>
       <limit lower="${radians(-350)}" upper="${radians(350)}" effort="0" velocity="${radians(219)}"/>
     </joint>
