Commit message: Update blender

File: kuka_kr20_support/urdf/kr20r1810_2.xacro (robot description, xacro)
@@ -1,4 +1,4 @@
 <?xml version="1.0"?>
-<robot name="kuka_kr20"
+<robot name="kr20r1810_2"
   xmlns:xacro="http://wiki.ros.org/xacro">
   <xacro:include filename="$(find kuka_kr20_support)/urdf/kr20r1810_2_macro.xacro"/>

File: kuka_kr20_support/urdf/kr20r1810_2_macro.xacro (robot description, xacro)
@@ -29,5 +29,5 @@
             <parent link="${prefix}base_link" />
             <child link="${prefix}link_1" />
-            <origin rpy="0.0 -0.0 0.0" xyz="0.0 0.0 0.2799999713897705" />
+            <origin rpy="0.0 -0.0 0.0" xyz="0.0 0.0 0.28" />
             <axis xyz="0 0 -1"/>
             <limit lower="${radians(-185)}" upper="${radians(185)}" effort="0" velocity="${radians(200)}"/>
@@ -48,5 +48,5 @@
             <parent link="${prefix}link_1" />
             <child link="${prefix}link_2" />
-            <origin rpy="-0.0 1.570796251296997 0.0" xyz="0.15999996662139893 0.0 0.2399999499320984" />
+            <origin xyz="0.16 0.0 0.24" rpy="0.0 -0.0 0.0" />
             <axis xyz="0 1 0"/>
             <limit lower="${radians(-185)}" upper="${radians(65)}" effort="0" velocity="${radians(175)}"/>
@@ -67,5 +67,5 @@
             <parent link="${prefix}link_2" />
             <child link="${prefix}link_3" />
-            <origin rpy="-0.0 -1.570796251296997 0.0" xyz="-7.087962217156019e-09 0.0 0.7799994945526123" />
+            <origin xyz="0.78 0.0 0.0" rpy="0.0 0.0 0.0" />
             <axis xyz="0 1 0"/>
             <limit lower="${radians(-138)}" upper="${radians(175)}" effort="0" velocity="${radians(190)}"/>
@@ -86,5 +86,5 @@
             <parent link="${prefix}link_3" />
             <child link="${prefix}link_4" />
-            <origin rpy="0.0 -0.0 0.0" xyz="0.29999905824661255 0.0 0.15000009536743164" />
+            <origin rpy="0.0 -0.0 0.0" xyz="0.3 0.0 0.15" />
             <axis xyz="-1 0 0"/>
             <limit lower="${radians(-350)}" upper="${radians(350)}" effort="0" velocity="${radians(430)}"/>
@@ -105,5 +105,5 @@
             <parent link="${prefix}link_4" />
             <child link="${prefix}link_5" />
-            <origin rpy="0.0 -0.0 0.0" xyz="0.5599991083145142 0.0 2.980231954552437e-07" />
+            <origin rpy="0.0 -0.0 0.0" xyz="0.56 0.0 0.0" />
             <axis xyz="0 1 0"/>
             <limit lower="${radians(-130)}" upper="${radians(130)}" effort="0" velocity="${radians(430)}"/>
@@ -124,5 +124,5 @@
             <parent link="${prefix}link_5" />
             <child link="${prefix}link_6" />
-            <origin rpy="0.0 -1.6940658945086007e-21 0.0" xyz="0.1529996395111084 0.0 1.7881390590446244e-07" />
+            <origin rpy="0.0 0.0 0.0" xyz="0.153 0.0 0.0" />
             <axis xyz="-1 0 0"/>
             <limit lower="${radians(-350)}" upper="${radians(350)}" effort="0" velocity="${radians(630)}"/>
